File: elec-thruster-control-board.kicad_sch (KiCad schematic)
At the start: 58 parts, among them J1 Conn_01x01, J10 Conn_01x01, J11 gp17-pwm0B, J12 gp2-pwm1A, J13 Conn_01x06, J14 Conn_01x01, J15 gp6-pwm3A, J16 gp8-pwm4A, J17 Conn_01x01, J18 gp19-pwm1B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

Commit message: Updated footprint to vertical JST Connector for PCB and Schematic  Please enter the commit message for your changes. Lines starting
Parts:
- J11, J12, J15, J16, J18, J19, J2, J20, J21, J5: footprint Connector_JST:JST_PH_S2B-PH-K_1x02_P2.00mm_Horizontal -> Connector_JST:JST_PH_B2B-PH-K_1x02_P2.00mm_Vertical
Changed lines of the file:
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@@
 			)
 		)
-		(property "Footprint" "Connector_JST:JST_PH_S2B-PH-K_1x02_P2.00mm_Horizontal"
+		(property "Footprint" "Connector_JST:JST_PH_B2B-PH-K_1x02_P2.00mm_Vertical"
 			(at 203.2 27.94 0)
 			(effects
@@
 			)
 		)
-		(property "Footprint" "Connector_JST:JST_PH_S2B-PH-K_1x02_P2.00mm_Horizontal"
+		(property "Footprint" "Connector_JST:JST_PH_B2B-PH-K_1x02_P2.00mm_Vertical"
 			(at 35.56 33.02 0)
 			(effects
@@
 			)
 		)
-		(property "Footprint" "Connector_JST:JST_PH_S2B-PH-K_1x02_P2.00mm_Horizontal"
+		(property "Footprint" "Connector_JST:JST_PH_B2B-PH-K_1x02_P2.00mm_Vertical"
 			(at 35.56 53.34 0)
 			(effects
@@
 			)
 		)
-		(property "Footprint" "Connector_JST:JST_PH_S2B-PH-K_1x02_P2.00mm_Horizontal"
+		(property "Footprint" "Connector_JST:JST_PH_B2B-PH-K_1x02_P2.00mm_Vertical"
 			(at 204.47 109.22 0)
 			(effects
@@
 			)
 		)
-		(property "Footprint" "Connector_JST:JST_PH_S2B-PH-K_1x02_P2.00mm_Horizontal"
+		(property "Footprint" "Connector_JST:JST_PH_B2B-PH-K_1x02_P2.00mm_Vertical"
 			(at 35.56 118.11 0)
 			(effects
@@
 			)
 		)
-		(property "Footprint" "Connector_JST:JST_PH_S2B-PH-K_1x02_P2.00mm_Horizontal"
+		(property "Footprint" "Connector_JST:JST_PH_B2B-PH-K_1x02_P2.00mm_Vertical"
 			(at 35.56 96.52 0)
 			(effects
@@
 			)
 		)
-		(property "Footprint" "Connector_JST:JST_PH_S2B-PH-K_1x02_P2.00mm_Horizontal"
+		(property "Footprint" "Connector_JST:JST_PH_B2B-PH-K_1x02_P2.00mm_Vertical"
 			(at 204.47 48.26 0)
 			(effects
@@
 			)
 		)
-		(property "Footprint" "Connector_JST:JST_PH_S2B-PH-K_1x02_P2.00mm_Horizontal"
+		(property "Footprint" "Connector_JST:JST_PH_B2B-PH-K_1x02_P2.00mm_Vertical"
 			(at 204.47 87.63 0)
 			(effects
@@
 			)
 		)
-		(property "Footprint" "Connector_JST:JST_PH_S2B-PH-K_1x02_P2.00mm_Horizontal"
+		(property "Footprint" "Connector_JST:JST_PH_B2B-PH-K_1x02_P2.00mm_Vertical"
 			(at 204.47 68.58 0)
 			(effects
@@
 			)
 		)
-		(property "Footprint" "Connector_JST:JST_PH_S2B-PH-K_1x02_P2.00mm_Horizontal"
+		(property "Footprint" "Connector_JST:JST_PH_B2B-PH-K_1x02_P2.00mm_Vertical"
 			(at 35.56 74.93 0)
 			(effects

Commit message: Nearly finalized design here.
Parts:
- removed J1, J10, J14, J17, J3, J4, J6, J7, J8, J9: Conn_01x01, Connector_PinHeader_2.54mm:PinHeader_1x01_P2.54mm_Vertical, symbol Connector_Generic:Conn_01x01
- removed J13: Conn_01x06, Connector_PinHeader_2.54mm:PinHeader_1x06_P2.54mm_Vertical, symbol Connector_Generic:Conn_01x06
- added J13: Conn_01x07, Connector_PinHeader_2.54mm:PinHeader_1x07_P2.54mm_Vertical, symbol Connector_Generic:Conn_01x07
- added J22, J24: Conn_01x06, Connector_PinHeader_2.54mm:PinHeader_1x06_P2.54mm_Vertical, symbol Connector_Generic:Conn_01x06
Connections:
- net GND: now also J13.7 (Pin_7), J22.1 (Pin_1), J24.1 (Pin_1)
- net gp0-pwm0A: now also J22.6 (Pin_6)
- net gp17-pwm0B: now also J24.2 (Pin_2)
- net gp19-pwm1B: now also J24.3 (Pin_3)
- net gp2-pwm1A: now also J22.5 (Pin_5)
- net gp21-pwm2B: now also J24.4 (Pin_4)
- net gp26-pwm5A: now also J24.5 (Pin_5)
- net gp27-pwm5B: now also J24.6 (Pin_6)
- net gp4-pwm2A: now also J22.4 (Pin_4)
- net gp6-pwm3A: now also J22.3 (Pin_3)
- net gp8-pwm4A: now also J22.2 (Pin_2)
- net at A1.17 (GPIO13), R16.2: now also J13.4 (Pin_4)
- net at A1.16 (GPIO12), R15.2: now also J13.3 (Pin_3)
- net at A1.14 (GPIO10), R13.2: now also J13.1 (Pin_1)
- net at A1.15 (GPIO11), R14.2: now also J13.2 (Pin_2)
- net at A1.19 (GPIO14), R12.2: now also J13.5 (Pin_5)
- net at A1.20 (GPIO15), R11.2: now also J13.6 (Pin_6)
Other:
- moved on the sheet: D1, D2, D3, D4, J11, J12, J15, J16, J18, J19, J2, J20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

Commit message: Updated footprints in the schematic and pcb design. Also cleaned up some of the routing.
Parts:
- D1, D10, D11, D12, D13, D14, D15, D16, D2, D3, D4, D5, D6, D7, D8, D9: footprint LED_SMD:LED_0805_2012Metric -> Imported Footprints:LED_APT2012LZGCK
Changed lines of the file:
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@@
 			)
 		)
-		(property "Footprint" "LED_SMD:LED_0805_2012Metric"
+		(property "Footprint" "Imported Footprints:LED_APT2012LZGCK"
 			(at 173.99 40.64 0)
 			(effects
@@
 			)
 		)
-		(property "Footprint" "LED_SMD:LED_0805_2012Metric"
+		(property "Footprint" "Imported Footprints:LED_APT2012LZGCK"
 			(at 173.99 60.96 0)
 			(effects
@@
 			)
 		)
-		(property "Footprint" "LED_SMD:LED_0805_2012Metric"
+		(property "Footprint" "Imported Footprints:LED_APT2012LZGCK"
 			(at 44.45 133.35 0)
 			(effects
@@
 			)
 		)
-		(property "Footprint" "LED_SMD:LED_0805_2012Metric"
+		(property "Footprint" "Imported Footprints:LED_APT2012LZGCK"
 			(at 175.26 110.49 0)
 			(effects
@@
 			)
 		)
-		(property "Footprint" "LED_SMD:LED_0805_2012Metric"
+		(property "Footprint" "Imported Footprints:LED_APT2012LZGCK"
 			(at 172.72 77.47 0)
 			(effects
@@
 			)
 		)
-		(property "Footprint" "LED_SMD:LED_0805_2012Metric"
+		(property "Footprint" "Imported Footprints:LED_APT2012LZGCK"
 			(at 48.26 176.53 0)
 			(effects
@@
 			)
 		)
-		(property "Footprint" "LED_SMD:LED_0805_2012Metric"
+		(property "Footprint" "Imported Footprints:LED_APT2012LZGCK"
 			(at 69.85 53.34 0)
 			(effects
@@
 			)
 		)
-		(property "Footprint" "LED_SMD:LED_0805_2012Metric"
+		(property "Footprint" "Imported Footprints:LED_APT2012LZGCK"
 			(at 68.58 33.02 0)
 			(effects
@@
 			)
 		)
-		(property "Footprint" "LED_SMD:LED_0805_2012Metric"
+		(property "Footprint" "Imported Footprints:LED_APT2012LZGCK"
 			(at 171.45 20.32 0)
 			(effects
@@
 			)
 		)
-		(property "Footprint" "LED_SMD:LED_0805_2012Metric"
+		(property "Footprint" "Imported Footprints:LED_APT2012LZGCK"
 			(at 67.31 118.11 0)
 			(effects
@@
 			)
 		)
-		(property "Footprint" "LED_SMD:LED_0805_2012Metric"
+		(property "Footprint" "Imported Footprints:LED_APT2012LZGCK"
 			(at 45.72 154.94 0)
 			(effects
@@
 			)
 		)
-		(property "Footprint" "LED_SMD:LED_0805_2012Metric"
+		(property "Footprint" "Imported Footprints:LED_APT2012LZGCK"
 			(at 48.26 165.1 0)
 			(effects
@@
 			)
 		)
-		(property "Footprint" "LED_SMD:LED_0805_2012Metric"
+		(property "Footprint" "Imported Footprints:LED_APT2012LZGCK"
 			(at 69.85 74.93 0)
 			(effects
@@
 			)
 		)
-		(property "Footprint" "LED_SMD:LED_0805_2012Metric"
+		(property "Footprint" "Imported Footprints:LED_APT2012LZGCK"
 			(at 48.26 186.69 0)
 			(effects
@@
 			)
 		)
-		(property "Footprint" "LED_SMD:LED_0805_2012Metric"
+		(property "Footprint" "Imported Footprints:LED_APT2012LZGCK"
 			(at 44.45 143.51 0)
 			(effects
@@
 			)
 		)
-		(property "Footprint" "LED_SMD:LED_0805_2012Metric"
+		(property "Footprint" "Imported Footprints:LED_APT2012LZGCK"
 			(at 68.58 96.52 0)
 			(effects

Commit message: The definitive final edition of our thruster control board.
Parts:
- added J1, J3: gp8-pwm4A, Connector_JST:JST_PH_B2B-PH-K_1x02_P2.00mm_Vertical, symbol Connector_Generic:Conn_01x02
- added R17, R18: R, Resistor_SMD:R_0805_2012Metric, symbol Device:R
- D1, D10, D11, D12, D13, D14, D15, D16, D2, D3, D4, D5, D6, D7, D8, D9: footprint Imported Footprints:LED_APT2012LZGCK -> myLibrary:LED_APT2012LZGCK
Connections:
- net GND: now also R11.1, J1.1 (Pin_1), J3.1 (Pin_1), R18.1
- net at A1.14 (GPIO10), J13.1 (Pin_1): now also R12.2, J3.2 (Pin_2), R18.2; no longer R13.2
- net at A1.19 (GPIO14), J13.5 (Pin_5): now also R13.2; no longer R12.2
- net at A1.20 (GPIO15), J13.6 (Pin_6), R11.2: now also J1.2 (Pin_2), R17.2
- net at D12.2 (A): now also R17.1; no longer R12.1
- net at D11.2 (A): now also R12.1; no longer R11.1
Other:
- moved on the sheet: D13, R13

Commit message: Work in progress for the final design revision
Parts:
- removed H1, H2, H3, H4: MountingHole, MountingHole:MountingHole_3.2mm_M3_DIN965_Pad, symbol Mechanical:MountingHole
Other:
- moved on the sheet: J3

Commit message: Made several changes to the board. Almost done just needs RC
Parts:
- removed A1: RaspberryPi_Pico, Module:RaspberryPi_Pico_Common_THT, symbol MCU_Module:RaspberryPi_Pico
- added J4, J6: Conn_01x20_Socket, Connector_PinSocket_2.54mm:PinSocket_1x20_P2.54mm_Vertical, symbol Connector:Conn_01x20_Socket
Connections:
- net GND: now also J4.13 (Pin_13), J4.18 (Pin_18), J4.3 (Pin_3), J4.8 (Pin_8), J6.13 (Pin_13), J6.18 (Pin_18), J6.3 (Pin_3), J6.8 (Pin_8)
- net gp0-pwm0A: now also J4.1 (Pin_1)
- net gp17-pwm0B: now also J6.19 (Pin_19)
- net gp19-pwm1B: now also J6.16 (Pin_16)
- net gp2-pwm1A: now also J4.4 (Pin_4)
- net gp21-pwm2B: now also J6.14 (Pin_14)
- net gp26-pwm5A: now also J6.10 (Pin_10)
- net gp27-pwm5B: now also J6.9 (Pin_9)
- net gp4-pwm2A: now also J4.6 (Pin_6)
- net gp6-pwm3A: now also J4.9 (Pin_9)
- net gp8-pwm4A: now also J4.11 (Pin_11)
- net at J13.4 (Pin_4), R16.2: now also J4.17 (Pin_17)
- net at R10.2: now also J6.20 (Pin_20)
- net at J13.3 (Pin_3), R15.2: now also J4.16 (Pin_16)
- net at R5.2: now also J4.12 (Pin_12)
- net at J1.2 (Pin_2), J13.6 (Pin_6), R11.2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: now also J4.20 (Pin_20)
- net at R4.2: now also J4.10 (Pin_10)
- net at J13.1 (Pin_1), J3.2 (Pin_2), R12.2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: now also J4.14 (Pin_14)
- net at J13.2 (Pin_2), R14.2: now also J4.15 (Pin_15)
- net at J13.5 (Pin_5), R13.2: now also J4.19 (Pin_19)
- net at R1.2: now also J4.2 (Pin_2)
- net at R6.2: now also J6.17 (Pin_17)
- net at R7.2: now also J6.15 (Pin_15)
- net at R8.2: now also J6.12 (Pin_12)
- net at R9.2: now also J6.7 (Pin_7)
- net at R2.2: now also J4.5 (Pin_5)
- net at R3.2: now also J4.7 (Pin_7)
Other:
- moved on the sheet: D6, D7, D8, D9, R6, R7, R8, R9
